Commit message: debut de la modelisation Gazebo. state publisher de base écrit mais pas encore testé. README de urdf_mode... est à jour

File: urdf_modelisation_octanis/urdf/octanis1.urdf (robot description, URDF)
Before this commit: robot Octanis1, 11 links, 10 joints
Links:
- added link world
- link axe_back_left: mass None -> 0.03; geometry collision box size=0.015 0.275 0.04; visual box size=0.015 0.275 0.04
- link axe_back_right: mass None -> 0.03; geometry collision box size=0.015 0.275 0.04; visual box size=0.015 0.275 0.04
- link axe_front_left: mass None -> 0.03; geometry collision box size=0.015 0.275 0.04; visual box size=0.015 0.275 0.04
- link axe_front_right: mass None -> 0.03; geometry collision box size=0.015 0.275 0.04; visual box size=0.015 0.275 0.04
- link base_link: mass 2500 -> 2.5; geometry collision box size=0.32 0.32 0.16; visual box size=0.32 0.32 0.16
- link wheel_back_left: mass None -> 0.02; geometry collision cylinder length=0.045 radius=0.08; visual cylinder length=0.045 radius=0.08
- link wheel_back_right: mass None -> 0.02; geometry collision cylinder length=0.045 radius=0.08; visual cylinder length=0.045 radius=0.08
- link wheel_front_left: mass None -> 0.02; geometry collision cylinder length=0.045 radius=0.08; visual cylinder length=0.045 radius=0.08
- link wheel_front_right: mass None -> 0.02; geometry collision cylinder length=0.045 radius=0.08; visual cylinder length=0.045 radius=0.08
Joints:
- joint joint_IMU: origin xyz=0 9 0 rpy=0 0 0 -> xyz=0 0.09 0 rpy=0 0 0
- joint joint_LIDAR: origin xyz=0 13 0 rpy=0 0 0 -> xyz=0 0.13 0 rpy=0 0 0
- joint joint_axe_back_left: origin xyz=-18.25 0 -2 rpy=-2.21 0 0 -> xyz=-0.1825 0 -0.02 rpy=-2.21 0 0
- joint joint_axe_back_right: origin xyz=18.25 0 -2 rpy=-2.21 0 0 -> xyz=0.1825 0 -0.02 rpy=-2.21 0 0
- joint joint_axe_front_left: origin xyz=-16.75 0 -2 rpy=-0.93 0 0 -> xyz=-0.1675 0 -0.02 rpy=-0.93 0 0
- joint joint_axe_front_right: origin xyz=16.75 0 -2 rpy=-0.93 0 0 -> xyz=0.1675 0 -0.02 rpy=-0.93 0 0
- joint joint_wheel_back_left: origin xyz=-3 25 0 rpy=2.21 0 0 -> xyz=-0.03 0.25 0 rpy=2.21 0 0
- joint joint_wheel_back_right: origin xyz=3 25 0 rpy=2.21 0 0 -> xyz=0.03 0.25 0 rpy=2.21 0 0
- joint joint_wheel_front_left: origin xyz=-3 25 0 rpy=0.93 0 0 -> xyz=-0.03 0.25 0 rpy=0.93 0 0
- joint joint_wheel_front_right: origin xyz=3 25 0 rpy=0.93 0 0 -> xyz=0.03 0.25 0 rpy=0.93 0 0
