Commit message: Transformation into one clean workspace

File: catkin_ws/src/octanis1_description/urdf/octanis1.urdf (robot description, URDF)
Before this commit: robot Octanis1, 11 links, 10 joints
Links:
- removed link body
- added link base_link, mass 2.5; collision box size=0.32 0.32 0.16; visual box size=0.32 0.32 0.16
- link LIDAR: mass None -> 0.2; geometry visual cylinder length=0.06 radius=0.076
- link axe_back_left: mass None -> 0.3; geometry collision box size=0.015 0.275 0.04; visual box size=0.015 0.275 0.04
- link axe_back_right: mass None -> 0.3; geometry collision box size=0.015 0.275 0.04; visual box size=0.015 0.275 0.04
- link axe_front_left: mass None -> 0.3; geometry collision box size=0.015 0.275 0.04; visual box size=0.015 0.275 0.04
- link axe_front_right: mass None -> 0.3; geometry collision box size=0.015 0.275 0.04; visual box size=0.015 0.275 0.04
- link wheel_back_left: mass None -> 0.2; geometry collision cylinder length=0.045 radius=0.08; visual cylinder length=0.045 radius=0.08
- link wheel_back_right: mass None -> 0.2; geometry collision cylinder length=0.045 radius=0.08; visual cylinder length=0.045 radius=0.08
- link wheel_front_left: mass None -> 0.2; geometry collision cylinder length=0.045 radius=0.08; visual cylinder length=0.045 radius=0.08
- link wheel_front_right: mass None -> 0.2; geometry collision cylinder length=0.045 radius=0.08; visual cylinder length=0.045 radius=0.08
Joints:
- joint joint_IMU: origin xyz=0 9 0 rpy=0 0 0 -> xyz=0 0.09 0 rpy=0 0 0; parent body -> base_link
- joint joint_LIDAR: axis (none) -> 0 0 1; origin xyz=0 13 0 rpy=0 0 0 -> xyz=0 0.12 0.04 rpy=-0.96 0 0; parent body -> base_link; type fixed -> continuous
- joint joint_axe_back_left: origin xyz=-16 0 0 rpy=0 0 0 -> xyz=-0.1825 0 -0.02 rpy=-2.21 0 0; parent body -> base_link
- joint joint_axe_back_right: origin xyz=16 0 0 rpy=0 0 0 -> xyz=0.1825 0 -0.02 rpy=-2.21 0 0; parent body -> base_link
- joint joint_axe_front_left: origin xyz=-17.5 0 0 rpy=0 0 0 -> xyz=-0.1675 0 -0.02 rpy=-0.93 0 0; parent body -> base_link
- joint joint_axe_front_right: origin xyz=17.5 0 0 rpy=0 0 0 -> xyz=0.1675 0 -0.02 rpy=-0.93 0 0; parent body -> base_link
- joint joint_wheel_back_left: origin xyz=0 -17 -20 rpy=0 0 0 -> xyz=-0.03 0.25 0 rpy=2.21 0 0
- joint joint_wheel_back_right: origin xyz=0 -17 -20 rpy=0 0 0 -> xyz=0.03 0.25 0 rpy=2.21 0 0
- joint joint_wheel_front_left: origin xyz=0 17 -20 rpy=0 0 0 -> xyz=-0.03 0.25 0 rpy=0.93 0 0
- joint joint_wheel_front_right: origin xyz=0 17 -20 rpy=0 0 0 -> xyz=0.03 0.25 0 rpy=0.93 0 0

Commit message: adding lidar and bosch drivers, fixed frame publishing and ekf state estimation

File: catkin_ws/src/octanis1_description/urdf/octanis1.urdf (robot description, URDF)
Before this commit: robot octanis1, 11 links, 10 joints
Joints:
- joint joint_LIDAR: type continuous -> fixed

Commit message: fixing lidar frame

File: catkin_ws/src/octanis1_description/urdf/octanis1.urdf (robot description, URDF)
Before this commit: robot octanis1, 11 links, 10 joints
Joints:
- joint joint_LIDAR: axis 0 0 1 -> (none); origin xyz=0 0.12 0.04 rpy=-0.96 0 0 -> xyz=0 0.12 0.04 rpy=0 0.78 1.57

Commit message: add of the dGPS on the urdf representation and little modifications of coordinates in the file xacro

File: catkin_ws/src/octanis1_description/urdf/octanis1.urdf (robot description, URDF)
Before this commit: robot octanis1, 11 links, 10 joints
Links:
- added link dGPS, mass 0.1; visual cylinder length=0.1 radius=0.1
- link LIDAR: geometry visual cylinder length=0.04 radius=0.035
- link wheel_back_left: geometry collision cylinder length=0.045 radius=0.08; visual cylinder length=0.045 radius=0.075
- link wheel_back_right: geometry collision cylinder length=0.045 radius=0.075; visual cylinder length=0.045 radius=0.075
- link wheel_front_left: geometry collision cylinder length=0.045 radius=0.075; visual cylinder length=0.045 radius=0.075
- link wheel_front_right: geometry collision cylinder length=0.045 radius=0.075; visual cylinder length=0.045 radius=0.075
Joints:
- added joint joint_dGPS: type fixed, parent base_link, child dGPS, origin xyz=0 0.10 0.08 rpy=0 0 0
- joint joint_LIDAR: axis (none) -> 0 0 1; origin xyz=0 0.12 0.04 rpy=0 0.78 1.57 -> xyz=0 0.215 0.01 rpy=-0.96 0 0; type fixed -> continuous

File: catkin_ws/src/octanis1_description/urdf/octanis1.xacro (robot description, xacro)
@@ -4,11 +4,12 @@
 	<xacro:property name="name_robot" value="octanis1" />
 	<!-- POSITION CONSTANTS (only whose which can change) -->
-	<xacro:property name="length_LIDAR" value="0.06" />
-	<xacro:property name="radius_LIDAR" value="0.076" />
-	<xacro:property name="radius_wheel" value="0.08" />
+	<xacro:property name="length_LIDAR" value="0.04" />
+	<xacro:property name="radius_LIDAR" value="0.035" />
+	<xacro:property name="radius_wheel" value="0.075" />
 	<xacro:property name="length_wheel" value="0.045" />
 	<!-- INERTIAL CONSTANTS (because they can change) -->
 	<xacro:property name="weight_box" value="2.5" />
 	<xacro:property name="weight_LIDAR" value="0.2" />
+   <xacro:property name="weight_dGPS" value="0.1" />
 	<xacro:property name="weight_axe" value="0.3" />
 	<xacro:property name="weight_wheel" value="0.2" />
@@ -184,4 +185,14 @@
 		</visual>
 	</link>
+   <link name="dGPS">
+		<xacro:default_inertia mass="${weight_dGPS}"/>
+		<visual>
+			<origin xyz="0 0 0" rpy="0 0 0"/> <!-- angle de 55 = 0.96 rad-->
+			<geometry>
+				<cylinder length="0.1" radius="0.1"/>
+			</geometry>
+			<material name="black" />
+		</visual>
+	</link>
 	<link name="IMU" />
 	<joint name="joint_axe_front_left" type="continuous">
@@ -212,6 +223,11 @@
 		<parent link="base_link" />
 		<child link="LIDAR" />
-		<origin xyz="0 0.12 0.04" rpy="-0.96 0 0" />
+		<origin xyz="0 0.215 0.01" rpy="-0.96 0 0" />
 		<axis xyz="0 0 1" />
+	</joint>
+  <joint name="joint_dGPS" type="fixed">
+		<parent link="base_link" />
+		<child link="dGPS" />
+		<origin xyz="0 0.10 0.08" rpy="0 0 0" />
 	</joint>
 	<joint name="joint_IMU" type="fixed">
