Commit message: adding second imu frame

File: catkin_ws_mission/src/octanis1_description/urdf/octanis1.xacro (robot description, xacro)
@@ -196,4 +196,5 @@
 	</link>
 	<link name="IMU" />
+	<link name="IMU2" />
 	<joint name="joint_axe_front_left" type="continuous">
 		<parent link="base_link" />
@@ -235,4 +236,9 @@
 		<child link="IMU" />
 		<origin xyz="0 0.09 0" rpy="0 0 0" />
+	</joint>
+	<joint name="joint_IMU2" type="fixed">
+		<parent link="base_link" />
+		<child link="IMU2" />
+		<origin xyz="0 0.05 0" rpy="0 0 0" />
 	</joint>
 	<joint name="joint_wheel_front_left" type="continuous">
