Commit message: generating urdf from xacro

File: catkin_ws_mission/src/octanis1_description/urdf/octanis1.urdf (robot description, URDF)
Before this commit: robot octanis1, 12 links, 11 joints
Links:
- added link IMU2
Joints:
- added joint joint_IMU2: type fixed, parent base_link, child IMU2, origin xyz=0 0.05 0 rpy=0 0 0

Commit message: correcting lidar frame

File: catkin_ws_mission/src/octanis1_description/urdf/octanis1.urdf (robot description, URDF)
Before this commit: robot octanis1, 13 links, 12 joints
Joints:
- joint joint_LIDAR: axis 0 0 1 -> (none); origin xyz=0 0.215 0.01 rpy=-0.96 0 0 -> xyz=0 0.12 0.04 rpy=0 0.78 1.57; type continuous -> fixed

File: catkin_ws_mission/src/octanis1_description/urdf/octanis1.xacro (robot description, xacro)
@@ -185,5 +185,5 @@
 		</visual>
 	</link>
-   <link name="dGPS">
+        <link name="dGPS">
 		<xacro:default_inertia mass="${weight_dGPS}"/>
 		<visual>
@@ -221,11 +221,10 @@
 		<axis xyz="1 0 0" />
 	</joint>
-	<joint name="joint_LIDAR" type="continuous">
+	<joint name="joint_LIDAR" type="fixed">
 		<parent link="base_link" />
 		<child link="LIDAR" />
-		<origin xyz="0 0.215 0.01" rpy="-0.96 0 0" />
-		<axis xyz="0 0 1" />
-	</joint>
-  <joint name="joint_dGPS" type="fixed">
+		<origin rpy="0 0.78 1.57" xyz="0 0.12 0.04"/>
+	</joint>
+        <joint name="joint_dGPS" type="fixed">
 		<parent link="base_link" />
 		<child link="dGPS" />

Commit message: adding tf2_web_republisher for diagnostics website and removing old ekf config files

File: catkin_ws_mission/src/octanis1_description/urdf/octanis1.urdf (robot description, URDF)
Before this commit: robot octanis1, 13 links, 12 joints
Links:
- link LIDAR: geometry visual cylinder length=0.04 radius=0.1
- link dGPS: geometry 
Joints:
- joint joint_axe_back_left: type continuous -> fixed
- joint joint_axe_back_right: type continuous -> fixed
- joint joint_axe_front_left: type continuous -> fixed
- joint joint_axe_front_right: type continuous -> fixed
- joint joint_wheel_back_left: type continuous -> fixed
- joint joint_wheel_back_right: type continuous -> fixed
- joint joint_wheel_front_left: type continuous -> fixed
- joint joint_wheel_front_right: type continuous -> fixed

File: catkin_ws_mission/src/octanis1_description/urdf/octanis1.xacro (robot description, xacro)
@@ -5,5 +5,5 @@
 	<!-- POSITION CONSTANTS (only whose which can change) -->
 	<xacro:property name="length_LIDAR" value="0.04" />
-	<xacro:property name="radius_LIDAR" value="0.035" />
+	<xacro:property name="radius_LIDAR" value="0.1" />
 	<xacro:property name="radius_wheel" value="0.075" />
 	<xacro:property name="length_wheel" value="0.045" />
@@ -178,5 +178,5 @@
 		<xacro:default_inertia mass="${weight_LIDAR}"/>
 		<visual>
-			<origin xyz="0 0 0" rpy="0 0 0"/> <!-- angle de 55 = 0.96 rad-->
+			<origin rpy="0 0 0" xyz="0 0 0"/>
 			<geometry>
 				<cylinder length="${length_LIDAR}" radius="${radius_LIDAR}"/>
@@ -185,17 +185,10 @@
 		</visual>
 	</link>
-        <link name="dGPS">
+  <link name="dGPS">
 		<xacro:default_inertia mass="${weight_dGPS}"/>
-		<visual>
-			<origin xyz="0 0 0" rpy="0 0 0"/> <!-- angle de 55 = 0.96 rad-->
-			<geometry>
-				<cylinder length="0.1" radius="0.1"/>
-			</geometry>
-			<material name="black" />
-		</visual>
 	</link>
 	<link name="IMU" />
 	<link name="IMU2" />
-	<joint name="joint_axe_front_left" type="continuous">
+	<joint name="joint_axe_front_left" type="fixed">
 		<parent link="base_link" />
 		<child link="axe_front_left" />
@@ -203,5 +196,5 @@
 		<axis xyz="1 0 0" />
 	</joint>
-	<joint name="joint_axe_front_right" type="continuous">
+	<joint name="joint_axe_front_right" type="fixed">
 		<parent link="base_link" />
 		<child link="axe_front_right" />
@@ -209,5 +202,5 @@
 		<axis xyz="1 0 0" />
 	</joint>
-	<joint name="joint_axe_back_right" type="continuous">
+	<joint name="joint_axe_back_right" type="fixed">
 		<parent link="base_link" />
 		<child link="axe_back_right" />
@@ -215,5 +208,5 @@
 		<axis xyz="1 0 0" />
 	</joint>
-	<joint name="joint_axe_back_left" type="continuous">
+	<joint name="joint_axe_back_left" type="fixed">
 		<parent link="base_link" />
 		<child link="axe_back_left" />
@@ -226,5 +219,5 @@
 		<origin rpy="0 0.78 1.57" xyz="0 0.12 0.04"/>
 	</joint>
-        <joint name="joint_dGPS" type="fixed">
+  <joint name="joint_dGPS" type="fixed">
 		<parent link="base_link" />
 		<child link="dGPS" />
@@ -241,5 +234,5 @@
 		<origin xyz="0 0.05 0" rpy="0 0 0" />
 	</joint>
-	<joint name="joint_wheel_front_left" type="continuous">
+	<joint name="joint_wheel_front_left" type="fixed">
 		<parent link="axe_front_left" />
 		<child link="wheel_front_left" />
@@ -247,5 +240,5 @@
 		<axis xyz="1 0 0" />
 	</joint>
-	<joint name="joint_wheel_front_right" type="continuous">
+	<joint name="joint_wheel_front_right" type="fixed">
 		<parent link="axe_front_right" />
 		<child link="wheel_front_right" />
@@ -253,5 +246,5 @@
 		<axis xyz="1 0 0" />
 	</joint>
-	<joint name="joint_wheel_back_right" type="continuous">
+	<joint name="joint_wheel_back_right" type="fixed">
 		<parent link="axe_back_right" />
 		<child link="wheel_back_right" />
@@ -259,5 +252,5 @@
 		<axis xyz="1 0 0" />
 	</joint>
-	<joint name="joint_wheel_back_left" type="continuous">
+	<joint name="joint_wheel_back_left" type="fixed">
 		<parent link="axe_back_left" />
 		<child link="wheel_back_left" />

Commit message: adding small D to pidctrl, adjusting urdf to convention

File: catkin_ws_mission/src/octanis1_description/urdf/octanis1.urdf (robot description, URDF)
Before this commit: robot octanis1, 13 links, 12 joints
Links:
- link axe_back_left: geometry visual box size=0.275 0.015 0.04
- link axe_back_right: geometry visual box size=0.275 0.015 0.04
- link axe_front_left: geometry visual box size=0.275 0.015 0.04
- link axe_front_right: geometry visual box size=0.275 0.015 0.04
- link wheel_back_left: geometry visual cylinder length=0.045 radius=0.075
- link wheel_back_right: geometry visual cylinder length=0.045 radius=0.075
- link wheel_front_left: geometry visual cylinder length=0.045 radius=0.075
- link wheel_front_right: geometry visual cylinder length=0.045 radius=0.075
Joints:
- joint joint_IMU: origin xyz=0 0.09 0 rpy=0 0 0 -> xyz=0 0 -0.055 rpy=0 0 0
- joint joint_IMU2: origin xyz=0 0.05 0 rpy=0 0 0 -> xyz=0 0.08 -0.03 rpy=0 0 0
- joint joint_LIDAR: origin xyz=0 0.12 0.04 rpy=0 0.78 1.57 -> xyz=0.12 0.05 0.04 rpy=0 0.78 0
- joint joint_axe_back_left: axis 1 0 0 -> 0 1 0; origin xyz=-0.1825 0 -0.02 rpy=-2.21 0 0 -> xyz=0 -0.1675 -0.02 rpy=0 -0.78 0
- joint joint_axe_back_right: axis 1 0 0 -> 0 1 0; origin xyz=0.1825 0 -0.02 rpy=-2.21 0 0 -> xyz=0 0.1675 -0.02 rpy=0 -0.78 0
- joint joint_axe_front_left: axis 1 0 0 -> 0 1 0; origin xyz=-0.1675 0 -0.02 rpy=-0.93 0 0 -> xyz=0 -0.1675 -0.02 rpy=0 0.78 0
- joint joint_axe_front_right: axis 1 0 0 -> 0 1 0; origin xyz=0.1675 0 -0.02 rpy=-0.93 0 0 -> xyz=0 0.1675 -0.02 rpy=0 0.78 0
- joint joint_dGPS: origin xyz=0 0.10 0.08 rpy=0 0 0 -> xyz=-0.1 0 0.1 rpy=0 0 0
- joint joint_wheel_back_left: axis 1 0 0 -> 0 1 0; origin xyz=-0.03 0.25 0 rpy=2.21 0 0 -> xyz=-0.25 0 0 rpy=0 0 0
- joint joint_wheel_back_right: axis 1 0 0 -> 0 1 0; origin xyz=0.03 0.25 0 rpy=2.21 0 0 -> xyz=-0.25 0 0 rpy=0 0 0
- joint joint_wheel_front_left: axis 1 0 0 -> 0 1 0; origin xyz=-0.03 0.25 0 rpy=0.93 0 0 -> xyz=0.25 0 0 rpy=0 0 0
- joint joint_wheel_front_right: axis 1 0 0 -> 0 1 0; origin xyz=0.03 0.25 0 rpy=0.93 0 0 -> xyz=0.25 0 0 rpy=0 0 0

File: catkin_ws_mission/src/octanis1_description/urdf/octanis1.xacro (robot description, xacro)
@@ -35,6 +35,6 @@
 			</geometry>
 			<material name="yellow">
-        		<color rgba="0.97 0.79 0.2 1"/>
-        	</material>
+				<color rgba="0.97 0.79 0.2 1"/>
+			</material>
 		</visual>
 		<collision>
@@ -48,7 +48,7 @@
 		<xacro:default_inertia mass="${weight_axe}"/>
 		<visual>
-			<origin xyz="0 0.1175 -0.02" rpy="0 0 0"/>
-			<geometry>
-				<box size="0.015 0.275 0.04" />
+			<origin xyz="0.1375 0 0" rpy="0 0 0"/>
+			<geometry>
+				<box size="0.275 0.015 0.04" />
 			</geometry>
 			<material name="white">
@@ -56,122 +56,74 @@
         	</material>
 		</visual>
-		<collision>
-			<origin xyz="0 0.1175 -0.02" rpy="0 0 0"/>
-			<geometry>
-				<box size="0.015 0.275 0.04" />
-			</geometry>
-		</collision>
 	</link>
 	<link name="axe_front_right">
 		<xacro:default_inertia mass="${weight_axe}"/>
 		<visual>
-			<origin xyz="0 0.1175 -0.02" rpy="0 0 0"/>
-			<geometry>
-				<box size="0.015 0.275 0.04" />
-			</geometry>
-			<material name="white" />
-		</visual>
-		<collision>
-			<origin xyz="0 0.1175 -0.02" rpy="0 0 0"/>
-			<geometry>
-				<box size="0.015 0.275 0.04" />
-			</geometry>
-		</collision>
+			<origin xyz="0.1375 0 0" rpy="0 0 0"/>
+			<geometry>
+				<box size="0.275 0.015 0.04" />
+			</geometry>
+			<material name="white" />
+		</visual>
 	</link>
 	<link name="axe_back_right">
 		<xacro:default_inertia mass="${weight_axe}"/>
 		<visual>
-			<origin xyz="0 0.1175 -0.02" rpy="0 0 0"/>
-			<geometry>
-				<box size="0.015 0.275 0.04" />
-			</geometry>
-			<material name="white" />
-		</visual>
-		<collision>
-			<origin xyz="0 0.1175 -0.02" rpy="0 0 0"/>
-			<geometry>
-				<box size="0.015 0.275 0.04" />
-			</geometry>
-		</collision>
+			<origin xyz="-0.1375 0 0" rpy="0 0 0"/>
+			<geometry>
+				<box size="0.275 0.015 0.04" />
+			</geometry>
+			<material name="white" />
+		</visual>
 	</link>
 	<link name="axe_back_left">
 		<xacro:default_inertia mass="${weight_axe}"/>
 		<visual>
-			<origin xyz="0 0.1175 -0.02" rpy="0 0 0"/>
-			<geometry>
-				<box size="0.015 0.275 0.04" />
-			</geometry>
-			<material name="white" />
-		</visual>
-		<collision>
-			<origin xyz="0 0.1175 -0.02" rpy="0 0 0"/>
-			<geometry>
-				<box size="0.015 0.275 0.04" />
-			</geometry>
-		</collision>
+			<origin xyz="-0.1375 0 0" rpy="0 0 0"/>
+			<geometry>
+				<box size="0.275 0.015 0.04" />
+			</geometry>
+			<material name="white" />
+		</visual>
 	</link>
 	<link name="wheel_front_left">
 		<xacro:default_inertia mass="${weight_wheel}"/>
 		<visual>
-			<origin xyz="0 0 0" rpy="0 1.57 0"/>
-			<geometry>
-				<cylinder length="${length_wheel}" radius="${radius_wheel}"/>
-			</geometry>
-			<material name="white" />
-		</visual>
-		<collision>
-			<origin xyz="0 0 0" rpy="0 1.57 0"/>
-			<geometry>
-				<cylinder length="${length_wheel}" radius="${radius_wheel}"/>
-			</geometry>
-		</collision>
+			<origin xyz="0 0 0" rpy="1.57 0 0"/>
+			<geometry>
+				<cylinder length="${length_wheel}" radius="${radius_wheel}"/>
+			</geometry>
+			<material name="white" />
+		</visual>
 	</link>
 	<link name="wheel_front_right">
 		<xacro:default_inertia mass="${weight_wheel}"/>
 		<visual>
-			<origin xyz="0 0 0" rpy="0 1.57 0"/>
-			<geometry>
-				<cylinder length="${length_wheel}" radius="${radius_wheel}"/>
-			</geometry>
-			<material name="white" />
-		</visual>
-		<collision>
-			<origin xyz="0 0 0" rpy="0 1.57 0"/>
-			<geometry>
-				<cylinder length="${length_wheel}" radius="${radius_wheel}"/>
-			</geometry>
-		</collision>
+			<origin xyz="0 0 0" rpy="1.57 0 0"/>
+			<geometry>
+				<cylinder length="${length_wheel}" radius="${radius_wheel}"/>
+			</geometry>
+			<material name="white" />
+		</visual>
 	</link>
 	<link name="wheel_back_right">
 		<xacro:default_inertia mass="${weight_wheel}"/>
 		<visual>
-			<origin xyz="0 0 0" rpy="0 1.57 0"/>
-			<geometry>
-				<cylinder length="${length_wheel}" radius="${radius_wheel}"/>
-			</geometry>
-			<material name="white" />
-		</visual>
-		<collision>
-			<origin xyz="0 0 0" rpy="0 1.57 0"/>
-			<geometry>
-				<cylinder length="${length_wheel}" radius="${radius_wheel}"/>
-			</geometry>
-		</collision>
+			<origin xyz="0 0 0" rpy="1.57 0 0"/>
+			<geometry>
+				<cylinder length="${length_wheel}" radius="${radius_wheel}"/>
+			</geometry>
+			<material name="white" />
+		</visual>
 	</link>
 	<link name="wheel_back_left">
 		<xacro:default_inertia mass="${weight_wheel}"/>
 		<visual>
-			<origin xyz="0 0 0" rpy="0 1.57 0"/>
-			<geometry>
-				<cylinder length="${length_wheel}" radius="${radius_wheel}"/>
-			</geometry>
-			<material name="white" />
-		</visual>
-		<collision>
-			<origin xyz="0 0 0" rpy="0 1.57 0"/>
-			<geometry>
-				<cylinder length="${length_wheel}" radius="0.08"/>
-			</geometry>
-		</collision>
+			<origin xyz="0 0 0" rpy="1.57 0 0"/>
+			<geometry>
+				<cylinder length="${length_wheel}" radius="${radius_wheel}"/>
+			</geometry>
+			<material name="white" />
+		</visual>
 	</link>
 	<link name="LIDAR">
@@ -185,5 +137,5 @@
 		</visual>
 	</link>
-  <link name="dGPS">
+	<link name="dGPS">
 		<xacro:default_inertia mass="${weight_dGPS}"/>
 	</link>
@@ -193,68 +145,68 @@
 		<parent link="base_link" />
 		<child link="axe_front_left" />
-		<origin xyz="-0.1675 0 -0.02" rpy="-0.93 0 0" />
-		<axis xyz="1 0 0" />
+		<origin xyz="0 -0.1675 -0.02" rpy="0 0.78 0" />
+		<axis xyz="0 1 0" />
 	</joint>
 	<joint name="joint_axe_front_right" type="fixed">
 		<parent link="base_link" />
 		<child link="axe_front_right" />
-		<origin xyz="0.1675 0 -0.02" rpy="-0.93 0 0" />
-		<axis xyz="1 0 0" />
+		<origin xyz="0 0.1675 -0.02" rpy="0 0.78 0" />
+		<axis xyz="0 1 0" />
 	</joint>
 	<joint name="joint_axe_back_right" type="fixed">
 		<parent link="base_link" />
 		<child link="axe_back_right" />
-		<origin xyz="0.1825 0 -0.02" rpy="-2.21 0 0" />
-		<axis xyz="1 0 0" />
+		<origin xyz="0 0.1675 -0.02" rpy="0 -0.78 0" />
+		<axis xyz="0 1 0" />
 	</joint>
 	<joint name="joint_axe_back_left" type="fixed">
 		<parent link="base_link" />
 		<child link="axe_back_left" />
-		<origin xyz="-0.1825 0 -0.02" rpy="-2.21 0 0" />
-		<axis xyz="1 0 0" />
+		<origin xyz="0 -0.1675 -0.02" rpy="0 -0.78 0" />
+		<axis xyz="0 1 0" />
 	</joint>
 	<joint name="joint_LIDAR" type="fixed">
 		<parent link="base_link" />
 		<child link="LIDAR" />
-		<origin rpy="0 0.78 1.57" xyz="0 0.12 0.04"/>
-	</joint>
-  <joint name="joint_dGPS" type="fixed">
+		<origin rpy="0 0.78 0" xyz="0.12 0.05 0.04"/>
+	</joint>
+	<joint name="joint_dGPS" type="fixed">
 		<parent link="base_link" />
 		<child link="dGPS" />
-		<origin xyz="0 0.10 0.08" rpy="0 0 0" />
+		<origin xyz="-0.1 0 0.1" rpy="0 0 0" />
 	</joint>
 	<joint name="joint_IMU" type="fixed">
 		<parent link="base_link" />
 		<child link="IMU" />
-		<origin xyz="0 0.09 0" rpy="0 0 0" />
+		<origin xyz="0 0 -0.055" rpy="0 0 0" />
 	</joint>
 	<joint name="joint_IMU2" type="fixed">
 		<parent link="base_link" />
 		<child link="IMU2" />
-		<origin xyz="0 0.05 0" rpy="0 0 0" />
+		<origin xyz="0 0.08 -0.03" rpy="0 0 0" />
 	</joint>
 	<joint name="joint_wheel_front_left" type="fixed">
 		<parent link="axe_front_left" />
 		<child link="wheel_front_left" />
-		<origin xyz="-0.03 0.25 0" rpy="0.93 0 0" />
-		<axis xyz="1 0 0" />
+		<origin xyz="0.25 0 0" rpy="0 0 0" />
+		<axis xyz="0 1 0" />
 	</joint>
 	<joint name="joint_wheel_front_right" type="fixed">
 		<parent link="axe_front_right" />
 		<child link="wheel_front_right" />
-		<origin xyz="0.03 0.25 0" rpy="0.93 0 0" />
-		<axis xyz="1 0 0" />
+		<origin xyz="0.25 0 0" rpy="0 0 0" />
+		<axis xyz="0 1 0" />
 	</joint>
 	<joint name="joint_wheel_back_right" type="fixed">
 		<parent link="axe_back_right" />
 		<child link="wheel_back_right" />
-		<origin xyz="0.03 0.25 0" rpy="2.21 0 0" />
-		<axis xyz="1 0 0" />
+		<origin xyz="-0.25 0 0" rpy="0 0 0" />
+		<axis xyz="0 1 0" />
 	</joint>
 	<joint name="joint_wheel_back_left" type="fixed">
 		<parent link="axe_back_left" />
 		<child link="wheel_back_left" />
-		<origin xyz="-0.03 0.25 0" rpy="2.21 0 0" />
-		<axis xyz="1 0 0" />
+		<origin xyz="-0.25 0 0" rpy="0 0 0" />
+		<axis xyz="0 1 0" />
 	</joint>
 </robot>
